File: Combined_Common_Components_Pack/Optoelectronics.kicad_sch (KiCad schematic)
At the start: 7 parts, among them U6 PC817XI

Commit message: More circuits
Parts:
- added U19: MOC3021M, Package_DIP:SMDIP-6_W9.53mm, symbol Relay_SolidState:MOC3021M
- U6: Type SMD -> (none)
Other:
- moved on the sheet: D2, D21, D22, D23, D24, D4, U6

Commit message: Added some connectors and basic parts
Parts:
- added D41: LED_Dual_KAK, Library:LED_Dual_3227, symbol Symbols:LED_Dual
Changed lines of the file:
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@@
+	)
+	(symbol
+		(lib_id "Symbols:LED_Dual")
+		(at 123.19 38.1 0)
+		(mirror y)
+		(unit 1)
+		(exclude_from_sim no)
+		(in_bom yes)
+		(on_board yes)
+		(dnp no)
+		(property "Reference" "D41"
+			(at 121.3564 26.67 0)
+			(effects
+				(font
+					(size 1.27 1.27)
+				)
+			)
+		)
+		(property "Value" "LED_Dual_KAK"
+			(at 121.3564 29.21 0)
+			(effects
+				(font
+					(size 1.27 1.27)
+				)
+			)
+		)
+		(property "Footprint" "Library:LED_Dual_3227"
+			(at 121.666 48.006 0)
+			(effects
+				(font
+					(size 1.27 1.27)
+				)
+				(hide yes)
+			)
+		)
+		(property "Datasheet" "~"
+			(at 121.92 38.1 0)
+			(effects
+				(font
+					(size 1.27 1.27)
+				)
+				(hide yes)
+			)
+		)
+		(property "Description" "Red, Emerald Green 625nm 525nm LED Indication - Discrete 2.4V 3.4V SMD-4P,3.2x2.7mm"
+			(at 123.19 38.1 0)
+			(effects
+				(font
+					(size 1.27 1.27)
+				)
+				(hide yes)
+			)
+		)
+		(property "LCSC" "C965842"
+			(at 122.936 45.466 0)
+			(effects
+				(font
+					(size 1.27 1.27)
+				)
+				(hide yes)
+			)
+		)
+		(property "Manufacturer " "XINGLIGHT"
+			(at 123.19 38.1 0)
+			(effects
+				(font
+					(size 1.27 1.27)
+				)
+				(hide yes)
+			)
+		)
+		(property "Mfr. Part Number" "XL-3227SURUGC"
+			(at 123.19 38.1 0)
+			(effects
+				(font
+					(size 1.27 1.27)
+				)
+				(hide yes)
+			)
+		)
+		(property "Observations" "Accepts other suppliers"
+			(at 123.19 38.1 0)
+			(effects
+				(font
+					(size 1.27 1.27)
+				)
+				(hide yes)
+			)
+		)
+		(pin "3"
+		)
+		(pin "4"
+		)
+		(pin "2"
+		)
+		(pin "1"
+		)
+		(instances
+			(project "Combined_Common_Components_Pack"
+				(path "/59e42e8e-5444-465a-b7a8-ffbd342a8d49/fd287e52-5b2b-4aeb-b67f-74078d3063e1"
+					(reference "D41")
+					(unit 1)
+				)
+			)
+		)
 	)
 	(symbol

Commit message: Minor updates
Basically components annotation, and more basic parts added
Parts:
- added U3: LTV-817, Package_DIP:SMDIP-4_W9.53mm, symbol Isolator:PC817
- U2: renamed from U6; Observations Accepts other suppliers -> Extended
- renumbered D22 to D14, D4 to D15, D21 to D16, D23 to D17, D41 to D18, D2 to D19, D24 to D20, U19 to U1
Changed lines of the file:
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@@
 		(on_board yes)
 		(dnp no)
-		(property "Reference" "D4"
+		(property "Reference" "D15"
 			(at 81.788 33.274 90)
 			(effects
@@
 			(project "Combined_Common_Components_Pack"
 				(path "/59e42e8e-5444-465a-b7a8-ffbd342a8d49/fd287e52-5b2b-4aeb-b67f-74078d3063e1"
-					(reference "D4")
+					(reference "D15")
 					(unit 1)
 				)
@@
 		(lib_id "Isolator:PC817")
 		(at 41.91 53.34 0)
-		(mirror y)
 		(unit 1)
 		(exclude_from_sim no)
@@
 		(on_board yes)
 		(dnp no)
-		(fields_autoplaced yes)
-		(property "Reference" "U6"
+		(property "Reference" "U2"
 			(at 41.91 44.45 0)
 			(effects
@@
 		)
 		(property "Footprint" "Package_DIP:DIP-4_W8.89mm_SMDSocket_LongPads"
-			(at 46.99 58.42 0)
+			(at 36.83 58.42 0)
 			(effects
 				(font
@@
 			)
 		)
-		(property "Observations" "Accepts other suppliers"
-			(at 41.91 53.34 0)
-			(effects
-				(font
-					(size 1.27 1.27)
-				)
-				(hide yes)
+		(property "Observations" "Extended"
+			(at 41.656 58.42 0)
+			(effects
+				(font
+					(size 1.27 1.27)
+				)
 			)
 		)
@@
 			(project "Combined_Common_Components_Pack"
 				(path "/59e42e8e-5444-465a-b7a8-ffbd342a8d49/fd287e52-5b2b-4aeb-b67f-74078d3063e1"
-					(reference "U6")
+					(reference "U2")
 					(unit 1)
 				)
@@
 		(on_board yes)
 		(dnp no)
-		(property "Reference" "D23"
+		(property "Reference" "D17"
 			(at 102.108 33.02 90)
 			(effects
@@
 			(project "Combined_Common_Components_Pack"
 				(path "/59e42e8e-5444-465a-b7a8-ffbd342a8d49/fd287e52-5b2b-4aeb-b67f-74078d3063e1"
-					(reference "D23")
+					(reference "D17")
 					(unit 1)
 				)
@@
 		(on_board yes)
 		(dnp no)
-		(property "Reference" "D41"
+		(property "Reference" "D18"
 			(at 121.3564 26.67 0)
 			(effects
@@
 			(project "Combined_Common_Components_Pack"
 				(path "/59e42e8e-5444-465a-b7a8-ffbd342a8d49/fd287e52-5b2b-4aeb-b67f-74078d3063e1"
-					(reference "D41")
+					(reference "D18")
 					(unit 1)
 				)
@@
 		(on_board yes)
 		(dnp no)
-		(property "Reference" "D22"
+		(property "Reference" "D14"
 			(at 70.358 33.02 90)
 			(effects
@@
 			(project "Combined_Common_Components_Pack"
 				(path "/59e42e8e-5444-465a-b7a8-ffbd342a8d49/fd287e52-5b2b-4aeb-b67f-74078d3063e1"
-					(reference "D22")
+					(reference "D14")
 					(unit 1)
 				)
@@
 		(on_board yes)
 		(dnp no)
-		(property "Reference" "U19"
+		(property "Reference" "U1"
 			(at 41.91 29.718 0)
 			(effects
@@
 			(project "Combined_Common_Components_Pack"
 				(path "/59e42e8e-5444-465a-b7a8-ffbd342a8d49/fd287e52-5b2b-4aeb-b67f-74078d3063e1"
-					(reference "U19")
+					(reference "U1")
 					(unit 1)
 				)
@@
 		(on_board yes)
 		(dnp no)
-		(property "Reference" "D24"
+		(property "Reference" "D20"
 			(at 89.662 50.546 0)
 			(effects
@@
 			(project "Combined_Common_Components_Pack"
 				(path "/59e42e8e-5444-465a-b7a8-ffbd342a8d49/fd287e52-5b2b-4aeb-b67f-74078d3063e1"
-					(reference "D24")
+					(reference "D20")
+					(unit 1)
+				)
+			)
+		)
+	)
+	(symbol
+		(lib_id "Isolator:PC817")
+		(at 41.91 71.12 0)
+		(unit 1)
+		(exclude_from_sim no)
+		(in_bom yes)
+		(on_board yes)
+		(dnp no)
+		(property "Reference" "U3"
+			(at 41.91 62.23 0)
+			(effects
+				(font
+					(size 1.27 1.27)
+				)
+			)
+		)
+		(property "Value" "LTV-817"
+			(at 41.91 64.77 0)
+			(effects
+				(font
+					(size 1.27 1.27)
+				)
+			)
+		)
+		(property "Footprint" "Package_DIP:SMDIP-4_W9.53mm"
+			(at 36.83 76.2 0)
+			(effects
+				(font
+					(size 1.27 1.27)
+					(italic yes)
+				)
+				(justify left)
+				(hide yes)
+			)
+		)
+		(property "Datasheet" "https://br.mouser.com/datasheet/2/365/Sharpelectronics_08292023_73758-3310502.pdf"
+			(at 41.91 71.12 0)
+			(effects
+				(font
+					(size 1.27 1.27)
+				)
+				(justify left)
+				(hide yes)
+			)
+		)
+		(property "Description" "-30℃~+110℃ 1 1.2V 100mV@1mA,20mA 35V 3us 4us@2mA,100Ω 50% 50mA 50mA 5kV 600% 6V DC Phototransistor SMD-4P Transistor, Photovoltaic Output Optoisolators ROHS"
+			(at 41.91 71.12 0)
+			(effects
+				(font
+					(size 1.27 1.27)
+				)
+				(hide yes)
+			)
+		)
+		(property "Manufacturer " "Slkor"
+			(at 41.91 71.12 0)
+			(effects
+				(font
+					(size 1.27 1.27)
+				)
+				(hide yes)
+			)
+		)
+		(property "Mfr. Part Number" "PC817B"
+			(at 41.91 71.12 0)
+			(effects
+				(font
+					(size 1.27 1.27)
+				)
+				(hide yes)
+			)
+		)
+		(property "Observations" "Basic"
+			(at 41.91 76.454 0)
+			(effects
+				(font
+					(size 1.27 1.27)
+				)
+			)
+		)
+		(property "LCSC" "C109227"
+			(at 41.91 71.12 0)
+			(effects
+				(font
+					(size 1.27 1.27)
+				)
+				(hide yes)
+			)
+		)
+		(pin "1"
+		)
+		(pin "2"
+		)
+		(pin "3"
+		)
+		(pin "4"
+		)
+		(instances
+			(project "Combined_Common_Components_Pack"
+				(path "/59e42e8e-5444-465a-b7a8-ffbd342a8d49/fd287e52-5b2b-4aeb-b67f-74078d3063e1"
+					(reference "U3")
 					(unit 1)
 				)
@@
 		(on_board yes)
 		(dnp no)
-		(property "Reference" "D2"
+		(property "Reference" "D19"
 			(at 69.342 50.8 0)
 			(effects
@@
 			(project "Combined_Common_Components_Pack"
 				(path "/59e42e8e-5444-465a-b7a8-ffbd342a8d49/fd287e52-5b2b-4aeb-b67f-74078d3063e1"
-					(reference "D2")
+					(reference "D19")
 					(unit 1)
 				)
@@
 		(on_board yes)
 		(dnp no)
-		(property "Reference" "D21"
+		(property "Reference" "D16"
 			(at 91.948 33.274 90)
 			(effects
@@
 			(project "Combined_Common_Components_Pack"
 				(path "/59e42e8e-5444-465a-b7a8-ffbd342a8d49/fd287e52-5b2b-4aeb-b67f-74078d3063e1"
-					(reference "D21")
-					(unit 1)
-				)
+					(reference "D16")
+					(unit 1)
+				)
