File: Combined_Common_Components_Pack/Regulators.kicad_sch (KiCad schematic)
At the start: 65 parts, among them Q5 2N7002K, Q7 2N7002K, Q8 PMOS, U10 LM2596S-ADJ, U11 L78L05_SOT89, U12 XL6019, U3 TP5100, U4 TP4056, U5 XL4001, U7 AP2112K-3.3, U9 XL1509-5.0

Commit message: More circuits
Parts:
- added PS1: HLK-5M05, Converter_ACDC:Converter_ACDC_Hi-Link_HLK-5Mxx, symbol Converter_ACDC:HLK-5M05
- U3: Manufacturer TOPPOWER(南京拓微) -> (none); Supplier LCSC -> (none)
- U4: Manufacturer TPOWER(天源) -> (none); Supplier LCSC -> (none); Supplier Part C382139 -> (none)
- U5: Manufacturer XLSEMI(芯龙) -> (none); Supplier LCSC -> (none); Supplier Part C2988027 -> (none)
Connections:
- net +5V: now also PS1.4 (+Vout)
- net GND: now also C40.2, C41.2, U11.2 (GND), PS1.3 (-Vout)
- net CE renamed CS
- new net cold: PS1.2 (AC/N)
- new net hot: PS1.1 (AC/L)

Commit message: Minor updates
Basically components annotation, and more basic parts added
Parts:
- renumbered C22 to C23, C23 to C24, C24 to C25, C25 to C26, C26 to C27, C31 to C28, C32 to C29, C33 to C30, C34 to C31, C39 to C32, C40 to C33, C41 to C34, C27 to C35, C28 to C36, C45 to C37, C42 to C38, C43 to C39, C29 to C40, C30 to C41, D8 to D21, D9 to D22, D10 to D23, D18 to D24, D11 to D25, D12 to D26, D19 to D27, D13 to D28, F3 to F6, F4 to F7, L3 to L5, L1 to L6, L4 to L7, L2 to L8, Q5 to Q7, Q7 to Q9, R56 to R52, R57 to R53, R58 to R54, R59 to R55, R67 to R56, R60 to R57, R61 to R58, R62 to R59, R63 to R60, R76 to R61, R77 to R62, R64 to R63, R65 to R64, R66 to R65, R68 to R66, R69 to R67, R70 to R68, TP1 to TP2, U4 to U10, U5 to U11, U11 to U4, U7 to U5, U3 to U6, U9 to U7, U12 to U8, U10 to U9
Other:
- note added: "Hi-Link 220Vac to 5V"
- moved on the sheet: C28, C29, C30, C31, C32, C33, C34
