File: Combined_Common_Components_Pack/Transistors.kicad_sch (KiCad schematic)
At the start: 5 parts, among them Q1 BC817, Q2 2N7002K, Q3 BC807, Q4 PMOS, Q6 AO3400A

Commit message: Added some connectors and basic parts
Parts:
- added Q17: 2N7002K, Package_TO_SOT_SMD:SOT-23, symbol Transistor_FET:2N7002K
Other:
- note added: "Basic"
Changed lines of the file:
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@@
 	(generator_version "8.0")
 	(paper "A4")
+	(text "Basic"
+		(exclude_from_sim no)
+		(at 47.244 62.23 0)
+		(effects
+			(font
+				(size 1.27 1.27)
+			)
+		)
+	)
 	(symbol
 		(lib_id "Transistor_BJT:BC807")
@@
 					(unit 1)
 				)
+			)
+		)
+	)
+	(symbol
+		(lib_id "Transistor_FET:2N7002K")
+		(at 50.8 66.04 0)
+		(unit 1)
+		(exclude_from_sim no)
+		(in_bom yes)
+		(on_board yes)
+		(dnp no)
+		(property "Reference" "Q17"
+			(at 50.038 59.944 0)
+			(effects
+				(font
+					(size 1.27 1.27)
+				)
+				(justify left)
+			)
+		)
+		(property "Value" "2N7002K"
+			(at 56.896 71.628 90)
+			(effects
+				(font
+					(size 1.27 1.27)
+				)
+				(justify left)
+			)
+		)
+		(property "Footprint" "Package_TO_SOT_SMD:SOT-23"
+			(at 55.88 67.945 0)
+			(effects
+				(font
+					(size 1.27 1.27)
+					(italic yes)
+				)
+				(justify left)
+				(hide yes)
+			)
+		)
+		(property "Datasheet" "https://www.diodes.com/assets/Datasheets/ds30896.pdf"
+			(at 55.88 69.85 0)
+			(effects
+				(font
+					(size 1.27 1.27)
+				)
+				(justify left)
+				(hide yes)
+			)
+		)
+		(property "Description" "1 N-channel 115mA 2.5V 225mW 50pF 5pF 5Ω@10V 60V SOT-23 MOSFETs ROHS"
+			(at 50.8 66.04 0)
+			(effects
+				(font
+					(size 1.27 1.27)
+				)
+				(hide yes)
+			)
+		)
+		(property "LCSC" "C8545"
+			(at 50.8 66.04 0)
+			(effects
+				(font
+					(size 1.27 1.27)
+				)
+				(hide yes)
+			)
+		)
+		(property "ASSEMBLY" ""
+			(at 50.8 66.04 0)
+			(effects
+				(font
+					(size 1.27 1.27)
+				)
+				(hide yes)
+			)
+		)
+		(property "Observations" "60V 0.1A"
+			(at 58.674 67.31 90)
+			(effects
+				(font
+					(size 1.27 1.27)
+				)
+			)
+		)
+		(pin "1"
+		)
+		(pin "3"
+		)
+		(pin "2"
+		)
+		(instances
+			(project "Combined_Common_Components_Pack"
+				(path "/59e42e8e-5444-465a-b7a8-ffbd342a8d49/36bf7309-9fc3-46ce-8643-e60be50ac833"
+					(reference "Q17")
+					(unit 1)
+				)

Commit message: Minor updates
Basically components annotation, and more basic parts added
Parts:
- renumbered Q3 to Q1, Q4 to Q2, Q1 to Q3, Q2 to Q4, Q6 to Q5, Q17 to Q6
Changed lines of the file:
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@@
 		(on_board yes)
 		(dnp no)
-		(property "Reference" "Q3"
+		(property "Reference" "Q1"
 			(at 30.48 27.94 0)
 			(effects
@@
 			(project "Combined_Common_Components_Pack"
 				(path "/59e42e8e-5444-465a-b7a8-ffbd342a8d49/36bf7309-9fc3-46ce-8643-e60be50ac833"
-					(reference "Q3")
+					(reference "Q1")
 					(unit 1)
 				)
@@
 		(on_board yes)
 		(dnp no)
-		(property "Reference" "Q17"
+		(property "Reference" "Q6"
 			(at 50.038 59.944 0)
 			(effects
@@
 			(project "Combined_Common_Components_Pack"
 				(path "/59e42e8e-5444-465a-b7a8-ffbd342a8d49/36bf7309-9fc3-46ce-8643-e60be50ac833"
-					(reference "Q17")
+					(reference "Q6")
 					(unit 1)
 				)
@@
 		(on_board yes)
 		(dnp no)
-		(property "Reference" "Q6"
+		(property "Reference" "Q5"
 			(at 67.564 45.466 0)
 			(effects
@@
 			(project "Combined_Common_Components_Pack"
 				(path "/59e42e8e-5444-465a-b7a8-ffbd342a8d49/36bf7309-9fc3-46ce-8643-e60be50ac833"
-					(reference "Q6")
+					(reference "Q5")
 					(unit 1)
 				)
@@
 		(on_board yes)
 		(dnp no)
-		(property "Reference" "Q2"
+		(property "Reference" "Q4"
 			(at 50.038 43.434 0)
 			(effects
@@
 			(project "Combined_Common_Components_Pack"
 				(path "/59e42e8e-5444-465a-b7a8-ffbd342a8d49/36bf7309-9fc3-46ce-8643-e60be50ac833"
-					(reference "Q2")
+					(reference "Q4")
 					(unit 1)
 				)
@@
 		(on_board yes)
 		(dnp no)
-		(property "Reference" "Q1"
+		(property "Reference" "Q3"
 			(at 29.972 46.736 0)
 			(effects
@@
 			(project "Combined_Common_Components_Pack"
 				(path "/59e42e8e-5444-465a-b7a8-ffbd342a8d49/36bf7309-9fc3-46ce-8643-e60be50ac833"
-					(reference "Q1")
+					(reference "Q3")
 					(unit 1)
 				)
@@
 		(on_board yes)
 		(dnp no)
-		(property "Reference" "Q4"
+		(property "Reference" "Q2"
 			(at 47.752 34.29 90)
 			(effects
@@
 			(project "Combined_Common_Components_Pack"
 				(path "/59e42e8e-5444-465a-b7a8-ffbd342a8d49/36bf7309-9fc3-46ce-8643-e60be50ac833"
-					(reference "Q4")
+					(reference "Q2")
 					(unit 1)
 				)
