File: Combined_Common_Components_Pack/microcontrollers.kicad_sch (KiCad schematic)
At the start: 3 parts, among them U14 ESP32-WROVER-E, U15 ESP32-MINI-1, U16 ESP32-WROOM-32

Commit message: Minor updates
Basically components annotation, and more basic parts added
Parts:
- renumbered U14 to U19, U15 to U20, U16 to U21
Changed lines of the file:
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@@
 		(dnp no)
 		(fields_autoplaced yes)
-		(property "Reference" "U14"
+		(property "Reference" "U19"
 			(at 68.2341 16.51 0)
 			(effects
@@
 			(project "Combined_Common_Components_Pack"
 				(path "/59e42e8e-5444-465a-b7a8-ffbd342a8d49/cb13f388-8ee5-4775-ac76-d64bb37f3b9f"
-					(reference "U14")
+					(reference "U19")
 					(unit 1)
 				)
@@
 		(on_board yes)
 		(dnp no)
-		(property "Reference" "U16"
+		(property "Reference" "U21"
 			(at 238.506 26.924 0)
 			(effects
@@
 			(project "Combined_Common_Components_Pack"
 				(path "/59e42e8e-5444-465a-b7a8-ffbd342a8d49/cb13f388-8ee5-4775-ac76-d64bb37f3b9f"
-					(reference "U16")
+					(reference "U21")
 					(unit 1)
 				)
@@
 		(dnp no)
 		(fields_autoplaced yes)
-		(property "Reference" "#PWR97"
+		(property "Reference" "#PWR94"
 			(at 243.84 105.41 0)
 			(effects
@@
 			(project "Combined_Common_Components_Pack"
 				(path "/59e42e8e-5444-465a-b7a8-ffbd342a8d49/cb13f388-8ee5-4775-ac76-d64bb37f3b9f"
-					(reference "#PWR97")
+					(reference "#PWR94")
 					(unit 1)
 				)
@@
 		(on_board yes)
 		(dnp no)
-		(property "Reference" "#PWR76"
+		(property "Reference" "#PWR93"
 			(at 156.21 86.36 0)
 			(effects
@@
 			(project "Combined_Common_Components_Pack"
 				(path "/59e42e8e-5444-465a-b7a8-ffbd342a8d49/cb13f388-8ee5-4775-ac76-d64bb37f3b9f"
-					(reference "#PWR76")
+					(reference "#PWR93")
 					(unit 1)
 				)
@@
 		(on_board yes)
 		(dnp no)
-		(property "Reference" "#PWR75"
+		(property "Reference" "#PWR91"
 			(at 156.21 22.86 0)
 			(effects
@@
 			(project "Combined_Common_Components_Pack"
 				(path "/59e42e8e-5444-465a-b7a8-ffbd342a8d49/cb13f388-8ee5-4775-ac76-d64bb37f3b9f"
-					(reference "#PWR75")
+					(reference "#PWR91")
 					(unit 1)
 				)
@@
 		(dnp no)
 		(fields_autoplaced yes)
-		(property "Reference" "U15"
+		(property "Reference" "U20"
 			(at 158.4041 16.51 0)
 			(effects
@@
 			(project "Combined_Common_Components_Pack"
 				(path "/59e42e8e-5444-465a-b7a8-ffbd342a8d49/cb13f388-8ee5-4775-ac76-d64bb37f3b9f"
-					(reference "U15")
+					(reference "U20")
 					(unit 1)
 				)
@@
 		(on_board yes)
 		(dnp no)
-		(property "Reference" "#PWR73"
+		(property "Reference" "#PWR90"
 			(at 66.04 22.86 0)
 			(effects
@@
 			(project "Combined_Common_Components_Pack"
 				(path "/59e42e8e-5444-465a-b7a8-ffbd342a8d49/cb13f388-8ee5-4775-ac76-d64bb37f3b9f"
-					(reference "#PWR73")
+					(reference "#PWR90")
 					(unit 1)
 				)
@@
 		(on_board yes)
 		(dnp no)
-		(property "Reference" "#PWR74"
+		(property "Reference" "#PWR92"
 			(at 68.58 71.12 0)
 			(effects
@@
 			(project "Combined_Common_Components_Pack"
 				(path "/59e42e8e-5444-465a-b7a8-ffbd342a8d49/cb13f388-8ee5-4775-ac76-d64bb37f3b9f"
-					(reference "#PWR74")
+					(reference "#PWR92")
 					(unit 1)
 				)
