File: XL4001_Load_limiter/XL4001_Load_limiter/XL4001_Load_limiter.kicad_sch (KiCad schematic)
At the start: 28 parts, among them J1 5.08-2P-90, J2 5.08-2P-90, J3 Conn_01x02_Socket, Q1 PMOS, Q2 2N7002K, U1 XL4001

Commit message: Added base layout for Load Limiter
Parts:
- removed R8: 2.7k, Resistor_SMD:R_0805_2012Metric, symbol Device:R
- added H1, H2, H3, H4: MountingHole, MountingHole:MountingHole_3.2mm_M3, symbol Mechanical:MountingHole
- added RV1: 10k, Potentiometer_THT:Potentiometer_Runtron_RM-065_Vertical, symbol Device:R_Potentiometer_Trim
- R7: value 10k -> 8.2k; LCSC C17414 -> C17828; Mfr. Part Number 0805W8F1002T5E -> 0805W8F8201T5E
- U1: footprint Library:ESOP-8_L4.9-W3.9-P1.27-LS6.0-BL-EP -> Aleoexpress:ESOP-8_L4.9-W3.9-P1.27-LS6.0-BL-EP
- renumbered R9 to R8, R11 to R9
Connections:
- net FB_CH0: now also R7.2
- net PCH0: now also RV1.1, RV1.2; no longer R7.1
- new net: R7.1, RV1.3
Other:
- note added: "16.6V 1800mA CC Driver"
- note added: "VOUT=1.235*(1+RB/RA) 12.4 < VOUT < 21.0 9 < RB/RA < 16"
- note removed: "17V 1800mA CC Driver"
- note removed: "VOUT=1.235*(1+RB/RA) 17/1.235=(1+RB/RA) 12.77=RB/RA"

Commit message: Hotfixes
Parts:
- added D16: LED_GREEN, LED_SMD:LED_0805_2012Metric_Pad1.15x1.40mm_HandSolder, symbol Device:LED
- added R11: 8.2k, Resistor_SMD:R_0805_2012Metric, symbol Device:R
- D1: footprint Diode_SMD:D_SMC_Handsoldering -> Diode_SMD:D_SMA
Connections:
- net GND: now also R11.1
- net PCH0: now also D16.2 (A)
- new net: D16.1 (K), R11.2
